File: netzteil.brd (EAGLE design)
At the start: 100 x 80 mm, 61 parts, among them IC1 LM723N, IC2 TL072P, Q1 BC559A, X1 MKDSN1,5/3-5,08, X10 2N3055, X11 MKDSN1,5/3-5,08, X12 POWER_KO, X13 V+, X14 V-, X2 MKDSN1,5/2-5,08, X3 MKDSN1,5/2-5,08, X4 50k, X5 1k, X7 STROMMESSUNG, X8 2N3055, X9 2N3055

Commit message: added minimum temperature enable for fan, fixed errors in regulation, adapted clamps for panel meters, added C.V. and overtemperature display diode, seperate supply for fan
Parts:
- removed X12: POWER_KO, con-phoenix-508:MKDSN1,5/2-5,08
- added B1, B2: (no value), rectifier:2KBB
- added C12, C13: 100n, rcl:C025-025X050
- added C14: 10u, rcl:E3,5-8
- added C4, C5: 2200u/63V, rcl:E7,5-18
- added D10, D12, D9: 1N4148DO35-7, diode:DO35-7
- added D11, D13: 3v3, diode:DO34Z7
- added D8: 1N4004, adafruit:DO41-10
- added IC3: TL084P, linear:DIL14
- added IC4: UA741P, linear:DIL08
- added LED2, LED3: (no value), adafruit:LED3MM
- added Q2, Q3, Q4: BC559A, transistor-pnp:TO92-EBC
- added R27, R29, R30, R40: 0R22/4W, powerR:4W_RM15
- added R28, R36: 100k, rcl:RTRIM3296Y
- added R31: 10R, rcl:0207/2V
- added R32, R33, R35, R37, R38: 4k7, rcl:0207/2V
- added R34, R39: 470R/1W, rcl:0207/2V
- added T2: BD241, transistor:TO220V
- added T3, T4, T5, T6: BD243, transistor:TO220
- added X6: VPOWER, con-phoenix-508:MKDSN1,5/2-5,08
- C10: value 100p -> 56p
- D6: value (none) -> 3v3
- IC2: value TL072P -> UA741P
- R12: device rcl:0411/12 -> rcl:0207/10
- R13: value R22/3W -> 0R22/4W; device rcl:0411/12 -> powerR:4W_RM15
- R16: value 10R/1W -> 100k; device rcl:0411/12 -> rcl:RTRIM3296Y
- R17: value R22/3W -> 2k2; device rcl:0411/12 -> rcl:0207/2V
- R18: value R22/3W -> 560R; device rcl:0411/12 -> rcl:0207/2V
- R19: value R22/3W -> 4k7; device rcl:0411/12 -> rcl:0207/7
- R24: value 470k -> 4k7
- R25: value 10k -> 0R22/4W; device rcl:RTRIM3296Y -> powerR:4W_RM15
- R26: value 10k -> 4k7
- T1: value (none) -> BD243; device transistor-neu-to92:TO220 -> transistor:TO220
- X10: value 2N3055 -> FAN; device con-phoenix-508:MKDSN1,5/3-5,08 -> con-phoenix-508:MKDSN1,5/2-5,08
- X11: value MKDSN1,5/3-5,08 -> SHUNT; device con-phoenix-508:MKDSN1,5/3-5,08 -> con-phoenix-508:MKDSN1,5/2-5,08
- X2: value MKDSN1,5/2-5,08 -> Vmess
- X3: value MKDSN1,5/2-5,08 -> OUTPUTCAP
- X7: value STROMMESSUNG -> VFAN
- X9: value 2N3055 -> NTC; device con-phoenix-508:MKDSN1,5/3-5,08 -> nxs_con-misc:2_2.54MM
- moved X10 198.8 mm to (-104.1, 29.2), turned to 0 degrees
- moved R25 181.6 mm to (-94.0, 64.8), turned to 0 degrees
- moved R22 177.4 mm to (-96.5, 108.0), turned to 0 degrees
- moved R23 176.0 mm to (-102.9, 108.0), turned to 0 degrees
- moved LED1 173.0 mm to (-109.2, 113.0), turned to 0 degrees
- moved R17 172.3 mm to (-83.8, 108.0)
- moved X7 169.6 mm to (-90.2, 29.2)
- moved R24 169.3 mm to (-109.2, 108.0), turned to 0 degrees
- moved D6 167.9 mm to (-108.0, 100.3), turned to 0 degrees
- moved D7 160.9 mm to (-92.7, 83.8), turned to 0 degrees
- moved R20 158.9 mm to (-90.2, 108.0), flipped to the top, turned to 0 degrees
- moved R13 157.1 mm to (-69.8, 64.8)
- moved R12 153.8 mm to (-95.2, 113.0), turned to 0 degrees
- moved R19 151.7 mm to (-38.1, 119.4)
- moved X9 149.9 mm to (-57.1, 41.9), turned to 0 degrees
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Connections:
- new net N$30: R23.2, R6.1, X14.1, X4.1
- new net N$33: D10.C, R26.3, R32.2
- new net N$34: LED2.A, R34.1
- new net N$35: C16.+, X3.2
- new net N$36: D12.C, IC3.1, Q3.E
- new net N$37: Q3.C, R18.2
- new net N$38: D12.A, Q3.B, R35.1
- new net N$39: IC3.8, R35.2
- new net N$40: IC3.10, R36.2
- new net N$41: IC3.2, R16.2
- new net N$42: C12.1, IC3.6, R19.1
- new net N$43: IC3.13, IC3.14
- new net N$44: R18.1, T1.1
- new net N$45: IC3.5, R28.2
- new net N$46: D8.C, R16.1, T1.3, X10.1
- new net N$47: C12.2, D9.C, IC3.7, R37.2
- new net N$48: R17.2, R19.2, X9.2
- new net N$49: R31.2, T2.3, T3.1, T4.1, T5.1, T6.1
- new net N$50: R27.P$1, T3.3
- new net N$51: R29.P$1, T4.3
- new net N$52: R30.P$1, T5.3
- new net N$53: B2.AC1, X7.2
- new net N$54: B2.AC2, X7.1
- new net N$55: B2.+, C14.+, T1.2
- new net N$56: D13.C, Q4.B, R38.2
- new net N$57: D13.A, R37.1
- new net N$58: Q4.C, R39.2
- new net N$59: LED3.A, R39.1
- new net N$63: R40.P$1, T6.3
- net AGND: now also C4.-, C5.+, D10.A, IC3.12, LED2.K, LED3.K, R7.1; no longer C8.2, C9.1, R6.1, X2.2, X3.1, X4.1, X5.1
- net N$10: now also IC2.6, R24.2; no longer IC2.1
- net N$11: now also IC4.2; no longer IC2.6
- net N$12: now also IC4.3; no longer IC2.5
- net N$15: now also D9.A, T2.1, X8.2; no longer T1.1
- net N$16: now also IC4.6; no longer IC2.7
- net N$17: now also R13.P$1, R27.P$2, R29.P$2, R30.P$2, R31.1, R40.P$2, X11.1, X8.3; no longer R13.2, R16.1, R17.1, R18.1, R19.1, R25.1
- net N$18: now also R25.P$2, X2.1, X3.1; no longer C16.+, R13.1, R24.1, R25.3, X7.1
- net N$19: now also R13.P$2, R25.P$1, X11.2; no longer R25.2, X7.2
- net N$21: now also D11.C, Q2.B, R33.2; no longer R16.2, T1.3, X10.2, X8.2, X9.2
- net N$22: now also D11.A, R24.1; no longer R17.2, X10.3
- net N$23: now also B1.AC1, X1.3; no longer R18.2, X9.3
- net N$24: now also B1.AC2, X1.1; no longer R19.2, X8.3
- net N$25: now also Q2.C, R34.2; no longer R24.2, R26.2, R26.3
- net N$29: now also T2.2, T3.2, T4.2, T5.2, T6.2, X6.2; no longer T1.2, X10.1, X11.3, X12.2, X9.1
- net N$31: now also X2.2, X6.1; no longer R26.1, X11.1, X12.1
- net N$32: now also R26.2, X5.1; no longer R23.2, R7.1, X14.1
- net V+: now also B1.+, C13.1, C4.+, C9.1, IC2.7, IC3.3, IC3.4, IC3.9, IC4.7, Q2.E, Q4.E, R28.3, R33.1, R36.3, R38.1, X9.1; no longer IC2.8, X1.3, X3.2
- net V-: now also B1.-, B2.-, C13.2, C14.-, C5.-, C8.2, D8.A, IC3.11, IC4.4, R16.3, R17.1, R28.1, R32.1, R36.1, X10.2; no longer X1.1, X2.1
Routing:
- net AGND: track 238.8 -> 0.00 mm, vias 4 -> 0
- net N$29: track 164.1 -> 0.00 mm, vias 10 -> 0
- net N$17: track 158.3 -> 0.00 mm, vias 2 -> 0
- net V+: track 120.3 -> 0.00 mm, vias 4 -> 0
- net N$31: track 117.0 -> 0.00 mm
- net N$21: track 92.4 -> 0.00 mm, vias 2 -> 0
- net N$18: track 91.8 -> 0.00 mm
- net N$7: track 74.6 -> 0.00 mm, vias 2 -> 0
- net N$32: track 51.6 -> 0.00 mm, vias 4 -> 0
- net V-: track 51.0 -> 0.00 mm
- net N$3: track 50.2 -> 0.00 mm
- net N$30: track 39.8 -> 0.00 mm
- net N$15: track 37.7 -> 0.00 mm, vias 2 -> 0
- net N$9: track 36.5 -> 0.00 mm, vias 4 -> 0
- net N$6: track 26.2 -> 0.00 mm
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- removed copper zone on layer 16, net AGND
Other:
- board text removed: "Labornetzeil"
- board text removed: "stonetronics &Fritz Holzer April 2018"

Commit message: added amperemeter and shunt clamps, semi-final version of the schematic for the pcb
Parts:
- removed R25: 0R22/4W, powerR:4W_RM15
- added X12: AMETER, con-phoenix-508:MKDSN1,5/2-5,08
- C14: value 10u -> 1000u
- R13: value 0R22/4W -> 0R1/4W
- X2: value Vmess -> VMETER
Connections:
- net N$17: now also X12.2; no longer D7.A, R27.P$2, R29.P$2, R30.P$2, R31.1, R40.P$2, X8.3
- net N$18: now also R13.P$2, X11.2; no longer R25.P$2
- net N$19: now also D7.A, R27.P$2, R29.P$2, R30.P$2, R31.1, R40.P$2, X12.1, X8.3; no longer R13.P$2, R25.P$1, X11.2
- net N$48: now also IC3.3, IC3.9
- net V+: no longer IC3.3, IC3.9

Commit message: finished pre-final pcb layout
Parts:
- added C15: 100n, rcl:C025-025X050
- B1, B2: device rectifier:2KBB -> rectifier:1KAB
- C14: value 1000u -> 470u; device rcl:E3,5-8 -> rcl:E5-13
- C4, C5: value 2200u/63V -> 1000u/63V
- D1: device adafruit:DO41-10 -> diode:DO41-10
- D11, D13, D6: device diode:DO34Z7 -> diode:SHORTDIODE
- D12, D2, D3: value 1N4148DO35-7 -> 1N4148V; device diode:DO35-7 -> diode:SHORTDIODE
- X1: value MKDSN1,5/3-5,08 -> VCONTROL
- X9: device nxs_con-misc:2_2.54MM -> con-phoenix-508:MKDSN1,5/2-5,08
- moved X12 274.3 mm to (95.2, 50.8), turned to 270 degrees
- moved R40 233.1 mm to (48.3, 61.0)
- moved T6 220.8 mm to (24.1, 83.6)
- moved R23 216.4 mm to (90.2, 10.2), turned to 180 degrees
- moved R12 199.5 mm to (86.4, 30.5), turned to 90 degrees
- moved R37 195.1 mm to (43.2, 48.3), turned to 90 degrees
- moved LED1 187.7 mm to (57.8, 27.4), turned to 270 degrees
- moved R22 186.5 mm to (62.2, 10.2)
- moved X3 185.4 mm to (76.2, 3.81)
- moved D6 185.2 mm to (66.8, 39.1), turned to 180 degrees
- moved R24 181.6 mm to (57.3, 35.6), turned to 90 degrees
- moved D7 181.2 mm to (87.6, 66.0), turned to 270 degrees
- moved T2 179.1 mm to (87.6, 79.9)
- moved Q4 178.3 mm to (41.9, 37.1), turned to 180 degrees
- moved R38 176.3 mm to (39.9, 43.2)
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Connections:
- net N$7 renamed V723
- net AGND: now also IC3.3; no longer IC3.12
- net N$20: now also D6.K; no longer D6.C
- net N$21: now also D11.K; no longer D11.C
- net N$3: now also D2.K; no longer D2.C
- net N$36: now also D12.K, IC3.14; no longer D12.C, IC3.1
- net N$41: now also IC3.13; no longer IC3.2
- net N$43: now also IC3.1, IC3.2; no longer IC3.13, IC3.14
- net N$48: now also C15.1, IC3.12, X9.1; no longer IC3.3, X9.2
- net N$56: now also D13.K; no longer D13.C
- net N$8: now also D3.K; no longer D3.C
- net V+: now also X9.2; no longer X9.1
- net V-: now also C15.2
Routing:
- net V+: track 0.00 -> 250.4 mm, vias 0 -> 3
- net V-: track 0.00 -> 184.0 mm, vias 0 -> 4
- net AGND: track 0.00 -> 164.2 mm, vias 0 -> 1
- net N$29: track 0.00 -> 150.7 mm, vias 0 -> 5
- net V723: track 0.00 -> 133.1 mm
- net N$18: track 0.00 -> 90.5 mm, vias 0 -> 3
- net N$49: track 0.00 -> 83.0 mm
- net N$30: track 0.00 -> 79.3 mm
- net N$15: track 0.00 -> 79.0 mm
- net N$3: track 0.00 -> 77.8 mm
- net N$31: track 0.00 -> 71.1 mm
- net N$19: track 0.00 -> 68.9 mm
- net N$14: track 0.00 -> 67.1 mm
- net N$17: track 0.00 -> 63.9 mm
- net N$46: track 0.00 -> 49.1 mm
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
Commit message: moved mechanical to thingiverse
Parts:
- removed D10: 1N4148DO35-7, diode:DO35-7
- removed R32: 4k7, rcl:0207/2V
- added F1: FUSEPICOFUSE, fuse:PICOFUSE
- added F2: 50mA, fuse:PICOFUSE
- added R25: 1k, rcl:0207/2V
- added R41: 10k, rcl:0207/2V
- added TP1, TP2, TP3, TP4, TP5: TPPAD1-13, testpad:P1-13
- T1, T3, T4, T5, T6: device transistor:TO220 -> transistor:TO220V
- moved T1 3.68 mm to (12.7, 79.9)
- moved T3 3.68 mm to (76.2, 79.9)
- moved T4 3.68 mm to (64.8, 79.9)
- moved T5 3.68 mm to (35.6, 79.9)
- moved T6 3.68 mm to (24.1, 79.9)
- moved LED1 2.54 mm to (55.2, 27.4)
- moved LED3 2.54 mm to (45.1, 27.4)
- moved R31 2.54 mm to (55.9, 77.5)
- moved X1 1.02 mm to (4.83, 40.6)
- moved X10 1.02 mm to (4.83, 64.8)
- moved X7 1.02 mm to (4.83, 54.6)
- moved R18 0.64 mm to (16.1, 41.1)
- moved C16 0.51 mm to (94.9, 15.0), flipped to the top, turned to 0 degrees
- moved D8 0.38 mm to (10.5, 66.0)
Connections:
- new net N$60: F1.1, X13.2
- new net N$7: IC3.2, R25.2, R41.2
- net AGND: now also F1.2, TP2.TP; no longer D10.A, X13.2
- net N$15: now also TP3.TP
- net N$30: now also F2.1; no longer X14.1
- net N$33: now also IC3.1, R25.1; no longer D10.C, R32.2
- net N$43: now also F2.2, X14.1; no longer IC3.1, IC3.2
- net V+: now also TP5.TP
- net V-: now also TP4.TP; no longer R32.1
- net V723: now also R41.1, TP1.TP
Routing:
- net N$43: track 2.54 -> 71.7 mm
- net N$33: track 9.95 -> 45.4 mm, vias 0 -> 1
- net N$7: track 0.00 -> 34.3 mm, vias 0 -> 2
- net N$60: track 0.00 -> 12.9 mm
- net V+: track 250.4 -> 262.0 mm
- net V-: track 184.0 -> 174.5 mm, vias 4 -> 3
- net N$30: track 79.3 -> 87.8 mm
- net N$51: track 18.2 -> 12.6 mm
- net V723: track 133.1 -> 137.9 mm
- net N$15: track 79.0 -> 82.8 mm
- net N$49: track 83.0 -> 86.0 mm
- net N$28: track 9.96 -> 12.5 mm
- net N$52: track 11.3 -> 13.4 mm
- net N$3: track 77.8 -> 79.6 mm
- net N$29: track 150.7 -> 152.4 mm
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- added copper zone on layer 16, net AGND
- added copper zone on layer 1, net V+
Other:
- outline, holes or cut-outs redrawn
- board text added: "+"
- board text added: "-"
- board text added: "-FAN+"
- board text added: "12/12/18"
- board text added: "1K IPoti"
- board text added: "50k VPoti"
- board text added: "A.M.+ A.M.-"
- board text added: "C B E"
- board text added: "COUT"
- board text added: "NTC"
- board text added: "Rshunt"
- board text added: "TP1"
- board text added: "TP2"
- board text added: "TP3"
- board text added: "TP4"
- board text added: "TP5"
- board text added: "V - VSen-"
- board text added: "V.M."
- board text added: "VAC FAN"
- board text added: "VPower+"
- board text added: "VPower-"
- board text added: "VSen+ V+"
- board text added: "powerSupply"
- board text added: "stonetronics"
- board text added: "~15V"
- board text added: "~15V GND"

Commit message: update readme.md
Parts:
- F1: value FUSEPICOFUSE -> 50mA
